File: UG_Power-Input/UG_Power-Input.sch (KiCad schematic (older format))
At the start: 46 parts, among them J1 12V IN, J2 12V OUT, J3 5V OUT, U1 LM2679

Commit message: Changes to terminal blocks
Parts:
- removed J1: 12V IN, TerminalBlock_Phoenix:TerminalBlock_Phoenix_MKDS-1,5-2-5.08_1x02_P5.08mm_Horizontal, symbol Connector:Screw_Terminal_01x02
- removed J2: 12V OUT, TerminalBlock_Phoenix:TerminalBlock_Phoenix_MKDS-1,5-2-5.08_1x02_P5.08mm_Horizontal, symbol Connector:Screw_Terminal_01x02
- removed J3: 5V OUT, TerminalBlock_Phoenix:TerminalBlock_Phoenix_MKDS-1,5-2-5.08_1x02_P5.08mm_Horizontal, symbol Connector:Screw_Terminal_01x02
- added J1: 12V IN, TerminalBlock_Weidemueller:TerminalBlock_Weidemueller_LMF-1330180000_1x02_P5.00mm_Vertical, symbol External~Components:TerminalBlock_Weidemüller_LMF-1330180000_1x02_P5.00mm_Vert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
- added J2: 5V OUT, TerminalBlock_Weidemueller:TerminalBlock_Weidemueller_LMF-1330180000_1x02_P5.00mm_Vertical, symbol External~Components:TerminalBlock_Weidemüller_LMF-1330180000_1x02_P5.00mm_Vert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
- added J3: 12V OUT, TerminalBlock_Weidemueller:TerminalBlock_Weidemueller_LMF-1330180000_1x02_P5.00mm_Vertical, symbol External~Components:TerminalBlock_Weidemüller_LMF-1330180000_1x02_P5.00mm_Vert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
Connections:
- wire segments 131 -> 149
Other:
- moved on the sheet: F1, F2, H1, H2, H3, H4, R3
